File: BSPD/BSPD.kicad_sch (KiCad schematic)
At the start: 32 parts, among them Q3 PMOS, U1 LM339DR, U10 641964-1, U2 SN74LVC1G08DBVR, U3 NE555DR, U4 SN74LVC3G14DCUR, U5 SN74AC32DR, U6 SN74LVC1G08DBVR, U7 641964-1, U8 R-78E5.0-0.5, U9 641964-1

Commit message: Fixes to BSPD
Parts:
- removed Q3: PMOS, Package_TO_SOT_SMD:SOT-23, symbol Simulation_SPICE:PMOS
- removed R1: 10K, Resistor_SMD:R_1206_3216Metric, symbol Device:R_US
- added Q101: Q_PMOS_GSD, Package_TO_SOT_SMD:SOT-523, symbol Transistor_FET:Q_PMOS_GSD
- renumbered C3 to C101, C1 to C102, C9 to C103, C2 to C104, C11 to C105, C13 to C106, C14 to C107, C10 to C108, C12 to C109, H1 to H101, H2 to H102, H3 to H103, H4 to H104, R3 to R101, R4 to R102, R2 to R103, RV1 to RV101, RV2 to RV102, RV3 to RV103, RV4 to RV104, U7 to U101, U9 to U102, U8 to U103, U2 to U104, U1 to U105, U3 to U106, U4 to U107, U5 to U108, U6 to U109, U10 to U110
Connections:
- net +5V: now also Q101.3 (D)
- net BSPD_TO_FAULT: now also Q101.2 (S)
- net at U109.4 (Y): now also Q101.1 (G)
Other:
- moved on the sheet: C109
